Commit message: edge_cases_solved

File: src/gg_hex_description/meshes/robot.urdf.xacro (robot description, xacro)
@@ -1,1867 +1,2062 @@
 <?xml version="1.0"?>
 <robot name="gg_hex"  xmlns:xacro= "http://www.ros.org/wiki/xacro">
-<link name="gg_head">
-<visual>
-<origin xyz="0.023562198419735225219 0.060799695286904251179 0.055047203654799869987" rpy="1.6298183611939731641 -0.041056855101145567355 0.16375605659172978723" />
-<geometry>
-<mesh filename="file://$(find gg_hex_description)/meshes/part_1.stl"/>
-</geometry>
-<material name="part_1_material">
-<color rgba="0.43921568627450979783 0.47450980392156860699 0.50196078431372548323 1.0"/>
-</material>
-</visual>
-<collision>
-<origin xyz="0.023562198419735225219 0.060799695286904251179 0.055047203654799869987" rpy="1.6298183611939731641 -0.041056855101145567355 0.16375605659172978723" />
-<geometry>
-<mesh filename="file://$(find gg_hex_description)/meshes/part_1.stl"/>
-</geometry>
-</collision>
-<visual>
-<origin xyz="0.35883672673370803352 0.056023028175970587816 0.22450447391026467914" rpy="1.511774292395820174 0.041056855101145685316 -2.9778365969980629124" />
-<geometry>
-<mesh filename="file://$(find gg_hex_description)/meshes/mg995_v3.stl"/>
-</geometry>
-<material name="mg995_v3_material">
+<link name="assembly_1">
+<visual>
+<origin xyz="0.045230512338216677382 0.077728783732269268736 -0.039250402362663638911" rpy="1.2246956414114624767 0.60592940837604103432 -2.4353792449475792914" />
+<geometry>
+<mesh filename="file://$(find gg_hex_description)/meshes/142-63448-1gen_a00.step.stl"/>
+</geometry>
+<material name="142-63448-1gen_a00.step_material">
+<color rgba="0.098039215686274508443 0.098039215686274508443 0.098039215686274508443 1.0"/>
+</material>
+</visual>
+<collision>
+<origin xyz="0.045230512338216677382 0.077728783732269268736 -0.039250402362663638911" rpy="1.2246956414114624767 0.60592940837604103432 -2.4353792449475792914" />
+<geometry>
+<mesh filename="file://$(find gg_hex_description)/meshes/142-63448-1gen_a00.step.stl"/>
+</geometry>
+</collision>
+<visual>
+<origin xyz="-0.070115829933568435406 0.13675320576692995278 -0.04957165911679123349" rpy="-2.6808124763527656498 0.88381758875990279467 1.2705962665396794975" />
+<geometry>
+<mesh filename="file://$(find gg_hex_description)/meshes/document.stl"/>
+</geometry>
+<material name="document_material">
+<color rgba="0.98039215686274505668 0.71372549019607844922 0.0039215686274509803377 1.0"/>
+</material>
+</visual>
+<collision>
+<origin xyz="-0.070115829933568435406 0.13675320576692995278 -0.04957165911679123349" rpy="-2.6808124763527656498 0.88381758875990279467 1.2705962665396794975" />
+<geometry>
+<mesh filename="file://$(find gg_hex_description)/meshes/document.stl"/>
+</geometry>
+</collision>
+<visual>
+<origin xyz="-0.13112567041683825808 0.10445699807928360281 0.0070111648683007232741" rpy="-1.2443384014361451584 -0.61573633691904516851 0.740458441131276901" />
+<geometry>
+<mesh filename="file://$(find gg_hex_description)/meshes/1side_2.stl"/>
+</geometry>
+<material name="1side_2_material">
+<color rgba="0.79215686274509800047 0.81960784313725487671 0.92941176470588238168 1.0"/>
+</material>
+</visual>
+<collision>
+<origin xyz="-0.13112567041683825808 0.10445699807928360281 0.0070111648683007232741" rpy="-1.2443384014361451584 -0.61573633691904516851 0.740458441131276901" />
+<geometry>
+<mesh filename="file://$(find gg_hex_description)/meshes/1side_2.stl"/>
+</geometry>
+</collision>
+<visual>
+<origin xyz="0.046300363008114575614 0.075117199756388142173 -0.039084188805817099421" rpy="1.2246956414114618106 0.60592940837604103432 -2.4353792449475792914" />
+<geometry>
+<mesh filename="file://$(find gg_hex_description)/meshes/porg_heat_sink.step.stl"/>
+</geometry>
+<material name="porg_heat_sink.step_material">
+<color rgba="0.098039215686274508443 0.098039215686274508443 0.098039215686274508443 1.0"/>
+</material>
+</visual>
+<collision>
+<origin xyz="0.046300363008114575614 0.075117199756388142173 -0.039084188805817099421" rpy="1.2246956414114618106 0.60592940837604103432 -2.4353792449475792914" />
+<geometry>
+<mesh filename="file://$(find gg_hex_description)/meshes/porg_heat_sink.step.stl"/>
+</geometry>
+</collision>
+<visual>
+<origin xyz="-0.030144414000453312319 0.11397461894422122874 0.069747045386147177304" rpy="-0.2234419486325698867 0.65516982812610802256 -2.2278876224107340143" />
+<geometry>
+<mesh filename="file://$(find gg_hex_description)/meshes/part_1.stl"/>
+</geometry>
+<material name="part_1_material">
+<color rgba="1 0.56862745098039213509 0.43529411764705883137 1.0"/>
+</material>
+</visual>
+<collision>
+<origin xyz="-0.030144414000453312319 0.11397461894422122874 0.069747045386147177304" rpy="-0.2234419486325698867 0.65516982812610802256 -2.2278876224107340143" />
+<geometry>
+<mesh filename="file://$(find gg_hex_description)/meshes/part_1.stl"/>
+</geometry>
+</collision>
+<visual>
+<origin xyz="-0.13136769558164909655 0.027634610643736345903 -0.022436195410797499239" rpy="0.44998642790264892222 -0.53803995526323666887 0.51481937495892005074" />
+<geometry>
+<mesh filename="file://$(find gg_hex_description)/meshes/part_1.stl"/>
+</geometry>
+<material name="part_1_material">
+<color rgba="1 0.56862745098039213509 0.43529411764705883137 1.0"/>
+</material>
+</visual>
+<collision>
+<origin xyz="-0.13136769558164909655 0.027634610643736345903 -0.022436195410797499239" rpy="0.44998642790264892222 -0.53803995526323666887 0.51481937495892005074" />
+<geometry>
+<mesh filename="file://$(find gg_hex_description)/meshes/part_1.stl"/>
+</geometry>
+</collision>
+<visual>
+<origin xyz="-0.12829445257991187179 0.10934444779962271266 0.011526593046762623196" rpy="-1.2150804522784592887 -0.60082170482534402733 0.68926844131497766455" />
+<geometry>
+<mesh filename="file://$(find gg_hex_description)/meshes/1side_4.stl"/>
+</geometry>
+<material name="1side_4_material">
+<color rgba="0.79215686274509800047 0.81960784313725487671 0.92941176470588238168 1.0"/>
+</material>
+</visual>
+<collision>
+<origin xyz="-0.12829445257991187179 0.10934444779962271266 0.011526593046762623196" rpy="-1.2150804522784592887 -0.60082170482534402733 0.68926844131497766455" />
+<geometry>
+<mesh filename="file://$(find gg_hex_description)/meshes/1side_4.stl"/>
+</geometry>
+</collision>
+<visual>
+<origin xyz="-0.0027343924302309363661 -0.072615223221202951365 -0.069788767742349100409" rpy="0.20097297559656263077 -0.66142953455963326981 0.9504299157554351174" />
+<geometry>
+<mesh filename="file://$(find gg_hex_description)/meshes/part_1.stl"/>
+</geometry>
+<material name="part_1_material">
+<color rgba="1 0.56862745098039213509 0.43529411764705883137 1.0"/>
+</material>
+</visual>
+<collision>
+<origin xyz="-0.0027343924302309363661 -0.072615223221202951365 -0.069788767742349100409" rpy="0.20097297559656263077 -0.66142953455963326981 0.9504299157554351174" />
+<geometry>
+<mesh filename="file://$(find gg_hex_description)/meshes/part_1.stl"/>
+</geometry>
+</collision>
+<visual>
+<origin xyz="0.098488889150964764596 0.013724785079281931477 0.0223944730545954096" rpy="-0.46565889858728348738 0.52490413390991141895 -2.6576949745600830788" />
+<geometry>
+<mesh filename="file://$(find gg_hex_description)/meshes/part_1.stl"/>
+</geometry>
+<material name="part_1_material">
+<color rgba="1 0.56862745098039213509 0.43529411764705883137 1.0"/>
+</material>
+</visual>
+<collision>
+<origin xyz="0.098488889150964764596 0.013724785079281931477 0.0223944730545954096" rpy="-0.46565889858728348738 0.52490413390991141895 -2.6576949745600830788" />
+<geometry>
+<mesh filename="file://$(find gg_hex_description)/meshes/part_1.stl"/>
+</geometry>
+</collision>
+<visual>
+<origin xyz="-1.4987603452312112662 -0.18773248174587564563 0.32807494299820194605" rpy="0 -0 0" />
+<geometry>
+<mesh filename="file://$(find gg_hex_description)/meshes/servo_motor_35kg_motor.stl"/>
+</geometry>
+<material name="servo_motor_35kg_motor_material">
+<color rgba="0.78039215686274510109 0.76078431372549015776 0.74117647058823532547 1.0"/>
+</material>
+</visual>
+<collision>
+<origin xyz="-1.4987603452312112662 -0.18773248174587564563 0.32807494299820194605" rpy="0 -0 0" />
+<geometry>
+<mesh filename="file://$(find gg_hex_description)/meshes/servo_motor_35kg_motor.stl"/>
+</geometry>
+</collision>
+<visual>
+<origin xyz="0.045127629807789892968 0.07739633252672784014 -0.038826052482414941114" rpy="1.2246956414114631428 0.60592940837604103432 -2.4353792449475792914" />
+<geometry>
+<mesh filename="file://$(find gg_hex_description)/meshes/porg_hex_standoff.step.stl"/>
+</geometry>
+<material name="porg_hex_standoff.step_material">
+<color rgba="1 0.92941176470588238168 0.43137254901960786491 1.0"/>
+</material>
+</visual>
+<collision>
+<origin xyz="0.045127629807789892968 0.07739633252672784014 -0.038826052482414941114" rpy="1.2246956414114631428 0.60592940837604103432 -2.4353792449475792914" />
+<geometry>
+<mesh filename="file://$(find gg_hex_description)/meshes/porg_hex_standoff.step.stl"/>
+</geometry>
+</collision>
+<visual>
+<origin xyz="0.045249484116786586885 0.077790088509967436625 -0.039328653470318830632" rpy="1.2246956414114618106 0.60592940837604103432 -2.4353792449475792914" />
+<geometry>
+<mesh filename="file://$(find gg_hex_description)/meshes/porg_system_screw.step_3.stl"/>
+</geometry>
+<material name="porg_system_screw.step_3_material">
+<color rgba="0.96078431372549022438 0.96078431372549022438 0.96470588235294119084 1.0"/>
+</material>
+</visual>
+<collision>
+<origin xyz="0.045249484116786586885 0.077790088509967436625 -0.039328653470318830632" rpy="1.2246956414114618106 0.60592940837604103432 -2.4353792449475792914" />
+<geometry>
+<mesh filename="file://$(find gg_hex_description)/meshes/porg_system_screw.step_3.stl"/>
+</geometry>
+</collision>
+<visual>
+<origin xyz="-0.12930566221565625851 0.10899780516645840578 0.011009855379071453729" rpy="-1.2246956414114613665 -0.60592940837604103432 0.70621340864221371358" />
+<geometry>
+<mesh filename="file://$(find gg_hex_description)/meshes/1side.stl"/>
+</geometry>
+<material name="1side_material">
+<color rgba="0.79215686274509800047 0.81960784313725487671 0.92941176470588238168 1.0"/>
+</material>
+</visual>
+<collision>
+<origin xyz="-0.12930566221565625851 0.10899780516645840578 0.011009855379071453729" rpy="-1.2246956414114613665 -0.60592940837604103432 0.70621340864221371358" />
+<geometry>
+<mesh filename="file://$(find gg_hex_description)/meshes/1side.stl"/>
+</geometry>
+</collision>
+<visual>
+<origin xyz="0.045249484116786586885 0.077790088509967436625 -0.039328653470318830632" rpy="1.2246956414114618106 0.60592940837604103432 -2.4353792449475792914" />
+<geometry>
+<mesh filename="file://$(find gg_hex_description)/meshes/porg_system_screw.step_2.stl"/>
+</geometry>
+<material name="porg_system_screw.step_2_material">
+<color rgba="0.96078431372549022438 0.96078431372549022438 0.96470588235294119084 1.0"/>
+</material>
+</visual>
+<collision>
+<origin xyz="0.045249484116786586885 0.077790088509967436625 -0.039328653470318830632" rpy="1.2246956414114618106 0.60592940837604103432 -2.4353792449475792914" />
+<geometry>
+<mesh filename="file://$(find gg_hex_description)/meshes/porg_system_screw.step_2.stl"/>
+</geometry>
+</collision>
+<visual>
+<origin xyz="0.04139700520505973369 0.077883349193068274197 -0.036722091151921820718" rpy="1.2246956414114624767 0.60592940837604103432 -2.4353792449475792914" />
+<geometry>
+<mesh filename="file://$(find gg_hex_description)/meshes/080-1656-000_3.step.stl"/>
+</geometry>
+<material name="080-1656-000_3.step_material">
+<color rgba="0.34901960784313723618 0.34901960784313723618 0.34901960784313723618 1.0"/>
+</material>
+</visual>
+<collision>
+<origin xyz="0.04139700520505973369 0.077883349193068274197 -0.036722091151921820718" rpy="1.2246956414114624767 0.60592940837604103432 -2.4353792449475792914" />
+<geometry>
+<mesh filename="file://$(find gg_hex_description)/meshes/080-1656-000_3.step.stl"/>
+</geometry>
+</collision>
+<visual>
+<origin xyz="0.045421954831058708457 0.078347404670860432141 -0.040040027176275028165" rpy="1.2246956414114633649 0.60592940837604103432 -2.4353792449475792914" />
+<geometry>
+<mesh filename="file://$(find gg_hex_description)/meshes/porg_system_screw.step_1.stl"/>
+</geometry>
+<material name="porg_system_screw.step_1_material">
+<color rgba="0.96078431372549022438 0.96078431372549022438 0.96470588235294119084 1.0"/>
+</material>
+</visual>
+<collision>
+<origin xyz="0.045421954831058708457 0.078347404670860432141 -0.040040027176275028165" rpy="1.2246956414114633649 0.60592940837604103432 -2.4353792449475792914" />
+<geometry>
+<mesh filename="file://$(find gg_hex_description)/meshes/porg_system_screw.step_1.stl"/>
+</geometry>
+</collision>
+<visual>
+<origin xyz="-0.13036098899584255828 0.10691828559453103731 0.0091248224959748491791" rpy="-1.2344489112767884631 -0.61090175020795234317 0.72327713354219846931" />
+<geometry>
+<mesh filename="file://$(find gg_hex_description)/meshes/1side_1.stl"/>
+</geometry>
+<material name="1side_1_material">
+<color rgba="0.79215686274509800047 0.81960784313725487671 0.92941176470588238168 1.0"/>
+</material>
+</visual>
+<collision>
+<origin xyz="-0.13036098899584255828 0.10691828559453103731 0.0091248224959748491791" rpy="-1.2344489112767884631 -0.61090175020795234317 0.72327713354219846931" />
+<geometry>
+<mesh filename="file://$(find gg_hex_description)/meshes/1side_1.stl"/>
+</geometry>
+</collision>
+<visual>
+<origin xyz="-0.12571212947564511242 0.1104013716602180728 0.012980703382802327717" rpy="-1.2056050252411003587 -0.59558105019003471092 0.67244322153912283735" />
+<geometry>
+<mesh filename="file://$(find gg_hex_description)/meshes/1side_3.stl"/>
+</geometry>
+<material name="1side_3_material">
+<color rgba="0.79215686274509800047 0.81960784313725487671 0.92941176470588238168 1.0"/>
+</material>
+</visual>
+<collision>
+<origin xyz="-0.12571212947564511242 0.1104013716602180728 0.012980703382802327717" rpy="-1.2056050252411003587 -0.59558105019003471092 0.67244322153912283735" />
+<geometry>
+<mesh filename="file://$(find gg_hex_description)/meshes/1side_3.stl"/>
+</geometry>
+</collision>
+<visual>
+<origin xyz="0.011598581326918544487 0.023763924025034188769 -0.033620637635183969749" rpy="-2.7954919682063597008 -0.60592940837604125637 0.70621340864221393563" />
+<geometry>
+<mesh filename="file://$(find gg_hex_description)/meshes/mounting_plate.step.stl"/>
+</geometry>
+<material name="mounting_plate.step_material">
 <color rgba="0.62745098039215685404 0.62745098039215685404 0.62745098039215685404 1.0"/>
 </material>
 </visual>
 <collision>
-<origin xyz="0.35883672673370803352 0.056023028175970587816 0.22450447391026467914" rpy="1.511774292395820174 0.041056855101145685316 -2.9778365969980629124" />
-<geometry>
-<mesh filename="file://$(find gg_hex_description)/meshes/mg995_v3.stl"/>
-</geometry>
-</collision>
-<visual>
-<origin xyz="0.067618785825018234981 0.0073717411514467668168 0.052932771556074148522" rpy="1.6298183611939731641 -0.041056855101145733888 0.16375605659173023132" />
-<geometry>
-<mesh filename="file://$(find gg_hex_description)/meshes/part_1.stl"/>
-</geometry>
-<material name="part_1_material">
-<color rgba="0.43921568627450979783 0.47450980392156860699 0.50196078431372548323 1.0"/>
-</material>
-</visual>
-<collision>
-<origin xyz="0.067618785825018234981 0.0073717411514467668168 0.052932771556074148522" rpy="1.6298183611939731641 -0.041056855101145733888 0.16375605659173023132" />
-<geometry>
-<mesh filename="file://$(find gg_hex_description)/meshes/part_1.stl"/>
-</geometry>
-</collision>
-<visual>
-<origin xyz="-0.36999161757788517901 -0.08448126780886903997 0.19285241442139863799" rpy="1.6298183611939731641 -0.041056855101145713072 0.16375605659173067541" />
-<geometry>
-<mesh filename="file://$(find gg_hex_description)/meshes/mg995_v3.stl"/>
-</geometry>
-<material name="mg995_v3_material">
+<origin xyz="0.011598581326918544487 0.023763924025034188769 -0.033620637635183969749" rpy="-2.7954919682063597008 -0.60592940837604125637 0.70621340864221393563" />
+<geometry>
+<mesh filename="file://$(find gg_hex_description)/meshes/mounting_plate.step.stl"/>
+</geometry>
+</collision>
+<visual>
+<origin xyz="0.045249484116786586885 0.077790088509967492136 -0.039328653470318886143" rpy="1.2246956414114618106 0.60592940837604103432 -2.4353792449475792914" />
+<geometry>
+<mesh filename="file://$(find gg_hex_description)/meshes/porg_hex_standoff.step_1.stl"/>
+</geometry>
+<material name="porg_hex_standoff.step_1_material">
+<color rgba="1 0.92941176470588238168 0.43137254901960786491 1.0"/>
+</material>
+</visual>
+<collision>
+<origin xyz="0.045249484116786586885 0.077790088509967492136 -0.039328653470318886143" rpy="1.2246956414114618106 0.60592940837604103432 -2.4353792449475792914" />
+<geometry>
+<mesh filename="file://$(find gg_hex_description)/meshes/porg_hex_standoff.step_1.stl"/>
+</geometry>
+</collision>
+<visual>
+<origin xyz="-0.13379184222027531992 0.10397273764580589051 0.0042527145773739727375" rpy="-1.2246956414114631428 -0.60592940837604125637 0.70621340864221393563" />
+<geometry>
+<mesh filename="file://$(find gg_hex_description)/meshes/cam_lider_stand.stl"/>
+</geometry>
+<material name="cam_lider_stand_material">
+<color rgba="0.79215686274509800047 0.81960784313725487671 0.93333333333333334814 1.0"/>
+</material>
+</visual>
+<collision>
+<origin xyz="-0.13379184222027531992 0.10397273764580589051 0.0042527145773739727375" rpy="-1.2246956414114631428 -0.60592940837604125637 0.70621340864221393563" />
+<geometry>
+<mesh filename="file://$(find gg_hex_description)/meshes/cam_lider_stand.stl"/>
+</geometry>
+</collision>
+<visual>
+<origin xyz="0.043263158096845555356 0.076507428087376594394 -0.037510805074619013588" rpy="1.2246956414114624767 0.60592940837604103432 -2.4353792449475792914" />
+<geometry>
+<mesh filename="file://$(find gg_hex_description)/meshes/142-13449-1000-a02.step.stl"/>
+</geometry>
+<material name="142-13449-1000-a02.step_material">
 <color rgba="0.62745098039215685404 0.62745098039215685404 0.62745098039215685404 1.0"/>
 </material>
 </visual>
 <collision>
-<origin xyz="-0.36999161757788517901 -0.08448126780886903997 0.19285241442139863799" rpy="1.6298183611939731641 -0.041056855101145713072 0.16375605659173067541" />
-<geometry>
-<mesh filename="file://$(find gg_hex_description)/meshes/mg995_v3.stl"/>
-</geometry>
-</collision>
-<visual>
-<origin xyz="-0.24881046969856607243 -0.1272813826038171614 0.059464627146769276356" rpy="3.1382040391284218295 -0.071804211987078134238 1.1746470986379109469" />
-<geometry>
-<mesh filename="file://$(find gg_hex_description)/meshes/part_3.stl"/>
-</geometry>
-<material name="part_3_material">
-<color rgba="0.26274509803921569651 0.28235294117647058432 0.30196078431372547213 1.0"/>
-</material>
-</visual>
-<collision>
-<origin xyz="-0.24881046969856607243 -0.1272813826038171614 0.059464627146769276356" rpy="3.1382040391284218295 -0.071804211987078134238 1.1746470986379109469" />
-<geometry>
-<mesh filename="file://$(find gg_hex_description)/meshes/part_3.stl"/>
-</geometry>
-</collision>
-<visual>
-<origin xyz="0.23820186996947737001 -0.29430221022616825932 0.19799079715707304516" rpy="1.5057047502754277168 -0.030523938227598110956 2.2603571641492261612" />
-<geometry>
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