Commit message: fix_complete_sim

File: install/gg_hex_description/share/gg_hex_description/simple_hex/robot.urdf.xacro (robot description, xacro)
@@ -18,7 +18,7 @@
 </collision>
 <inertial>
-<origin xyz="0 -1.3877787807814456755e-17 0.023199999999999998401" rpy="0 0 0"/>
+<origin xyz="0 -6.9388939039072283776e-18 0.023199999999999998401" rpy="0 0 0"/>
 <mass value="0.59529549486301092109" />
-<inertia ixx="0.0030748925185440610652" ixy="0"  ixz="0" iyy="0.0016906840458352412251" iyz="0" izz="0.0047035666169977386614" />
+<inertia ixx="0.0030748925185440614989" ixy="0"  ixz="0" iyy="0.0016906840458352414419" iyz="0" izz="0.0047035666169977386614" />
 </inertial>
 </link>
@@ -62,7 +62,7 @@
 </collision>
 <inertial>
-<origin xyz="0.0375016406817649528 2.7755575615628913511e-17 -0.002916799334743866174" rpy="0 0 0"/>
-<mass value="0.053756066729807983062" />
-<inertia ixx="6.1725657961057495281e-06" ixy="-3.9013430001076611365e-36"  ixz="4.0422270863664954962e-10" iyy="3.4211476506187116632e-05" iyz="4.0371463405644450255e-36" izz="3.3235315244488732836e-05" />
+<origin xyz="0.0375016406817649528 0 -0.0029167993347438657403" rpy="0 0 0"/>
+<mass value="0.053756066729807990001" />
+<inertia ixx="6.1725657961057495281e-06" ixy="-3.9013430001076611365e-36"  ixz="4.0422270863664960132e-10" iyy="3.4211476506187116632e-05" iyz="4.0371463405644450255e-36" izz="3.3235315244488732836e-05" />
 </inertial>
 </link>
@@ -84,7 +84,7 @@
 </collision>
 <inertial>
-<origin xyz="0.037500919815065446306 0 1.839630130919531673e-07" rpy="0 0 0"/>
-<mass value="0.053754736812063892704" />
-<inertia ixx="6.629807515216692076e-06" ixy="1.6458832113731393079e-38"  ixz="-5.3411963924549780679e-06" iyy="3.4666848127693282542e-05" iyz="-1.0240845939341500988e-37" izz="3.3233445124738763448e-05" />
+<origin xyz="0.037500919815065453244 0 1.8396301309196947268e-07" rpy="0 0 0"/>
+<mass value="0.053754736812063899642" />
+<inertia ixx="6.629807515216692076e-06" ixy="1.6458832113731393079e-38"  ixz="-5.3411963924549780679e-06" iyy="3.4666848127693275766e-05" iyz="-1.0240845939341500988e-37" izz="3.3233445124738763448e-05" />
 </inertial>
 </link>
@@ -106,7 +106,7 @@
 </collision>
 <inertial>
-<origin xyz="0.038984534277943398706 0 -0.0013659706120265349086" rpy="0 0 0"/>
+<origin xyz="0.038984534277943398706 0 -0.0013659706120265383781" rpy="0 0 0"/>
 <mass value="0.057365949134959140499" />
-<inertia ixx="6.7866051749620268655e-06" ixy="-2.3680935053173413778e-36"  ixz="-2.7857025297757682857e-06" iyy="3.6471388191653054305e-05" iyz="1.9541077328988703576e-35" izz="3.4867176458850274992e-05" />
+<inertia ixx="6.7866051749620268655e-06" ixy="-2.3680935053173413778e-36"  ixz="-2.7857025297757678622e-06" iyy="3.6471388191653054305e-05" iyz="1.9541077328988703576e-35" izz="3.4867176458850274992e-05" />
 </inertial>
 </link>
@@ -182,7 +182,7 @@
 </collision>
 <inertial>
-<origin xyz="0.037501640681764966678 2.7755575615628913511e-17 -0.0029167993347438449236" rpy="0 0 0"/>
-<mass value="0.053756066729807983062" />
-<inertia ixx="6.1725657961057495281e-06" ixy="0"  ixz="4.0422270863981537662e-10" iyy="3.4211476506187116632e-05" iyz="0" izz="3.3235315244488732836e-05" />
+<origin xyz="0.037501640681764966678 0 -0.0029167993347438449236" rpy="0 0 0"/>
+<mass value="0.053756066729807990001" />
+<inertia ixx="6.1725657961057495281e-06" ixy="0"  ixz="4.0422270863981542832e-10" iyy="3.4211476506187116632e-05" iyz="0" izz="3.3235315244488732836e-05" />
 </inertial>
 </link>
@@ -204,7 +204,7 @@
 </collision>
 <inertial>
-<origin xyz="0.037500919815065481 0 1.839630130957957852e-07" rpy="0 0 0"/>
-<mass value="0.053754736812063892704" />
-<inertia ixx="6.6298075152166937701e-06" ixy="0"  ixz="-5.3411963924549780679e-06" iyy="3.4666848127693282542e-05" iyz="0" izz="3.3233445124738763448e-05" />
+<origin xyz="0.037500919815065487939 0 1.8396301309581211706e-07" rpy="0 0 0"/>
+<mass value="0.053754736812063899642" />
+<inertia ixx="6.6298075152166937701e-06" ixy="0"  ixz="-5.3411963924549780679e-06" iyy="3.4666848127693275766e-05" iyz="0" izz="3.3233445124738763448e-05" />
 </inertial>
 </link>
@@ -226,7 +226,7 @@
 </collision>
 <inertial>
-<origin xyz="0.038984534277943565239 0 -0.0013659706120265173446" rpy="0 0 0"/>
+<origin xyz="0.038984534277943565239 0 -0.001365970612026520814" rpy="0 0 0"/>
 <mass value="0.057365949134959140499" />
-<inertia ixx="6.7866051749620285596e-06" ixy="-1.0663918689120664312e-36"  ixz="-2.7857025297757687092e-06" iyy="3.6471388191653054305e-05" iyz="1.3555009886619676805e-35" izz="3.4867176458850274992e-05" />
+<inertia ixx="6.7866051749620285596e-06" ixy="-1.0663918689120664312e-36"  ixz="-2.7857025297757682857e-06" iyy="3.6471388191653054305e-05" iyz="1.3555009886619676805e-35" izz="3.4867176458850274992e-05" />
 </inertial>
 </link>
@@ -302,7 +302,7 @@
 </collision>
 <inertial>
-<origin xyz="0.037501640681764973617 2.7755575615628913511e-17 -0.00291679933474384449" rpy="0 0 0"/>
-<mass value="0.053756066729807983062" />
-<inertia ixx="6.1725657961057495281e-06" ixy="3.3866754089596615417e-36"  ixz="4.042227086378962659e-10" iyy="3.4211476506187116632e-05" iyz="-4.9525034835553173072e-36" izz="3.3235315244488732836e-05" />
+<origin xyz="0.037501640681764980556 0 -0.0029167993347438440563" rpy="0 0 0"/>
+<mass value="0.053756066729807990001" />
+<inertia ixx="6.1725657961057495281e-06" ixy="3.3866754089596615417e-36"  ixz="4.042227086378963176e-10" iyy="3.4211476506187116632e-05" iyz="-4.9525034835553173072e-36" izz="3.3235315244488732836e-05" />
 </inertial>
 </link>
@@ -324,7 +324,7 @@
 </collision>
 <inertial>
-<origin xyz="0.037500919815065481 0 1.8396301310720860126e-07" rpy="0 0 0"/>
-<mass value="0.053754736812063892704" />
-<inertia ixx="6.629807515216692076e-06" ixy="8.4076706020862943724e-36"  ixz="-5.3411963924549780679e-06" iyy="3.4666848127693282542e-05" iyz="-5.2557119676207734611e-36" izz="3.3233445124738763448e-05" />
+<origin xyz="0.037500919815065487939 0 1.8396301310722493311e-07" rpy="0 0 0"/>
+<mass value="0.053754736812063899642" />
+<inertia ixx="6.629807515216692076e-06" ixy="8.4076706020862930361e-36"  ixz="-5.3411963924549780679e-06" iyy="3.4666848127693275766e-05" iyz="-5.2557119676207727929e-36" izz="3.3233445124738763448e-05" />
 </inertial>
 </link>
@@ -346,7 +346,7 @@
 </collision>
 <inertial>
-<origin xyz="0.038984534277943565239 0 -0.0013659706120265429317" rpy="0 0 0"/>
+<origin xyz="0.038984534277943565239 0 -0.0013659706120265464012" rpy="0 0 0"/>
 <mass value="0.057365949134959140499" />
-<inertia ixx="6.7866051749620285596e-06" ixy="1.1415885784153511439e-35"  ixz="-2.7857025297757674387e-06" iyy="3.6471388191653054305e-05" iyz="9.8847353391390472314e-36" izz="3.4867176458850274992e-05" />
+<inertia ixx="6.7866051749620285596e-06" ixy="1.1415885784153511439e-35"  ixz="-2.7857025297757670152e-06" iyy="3.6471388191653054305e-05" iyz="9.8847353391390472314e-36" izz="3.4867176458850274992e-05" />
 </inertial>
 </link>
@@ -385,5 +385,5 @@
 <link name="part_2_4">
 <visual>
-<origin xyz="1.3877787807814456755e-17 0 0.14999999999999999445" rpy="3.141592653589793116 -4.3645711874439094161e-32 -2.7440535728855418873e-17" />
+<origin xyz="1.3877787807814456755e-17 -1.3877787807814456755e-17 0.14999999999999999445" rpy="-3.141592653589793116 1.7984046345965779156e-32 3.88627629426162707e-17" />
 <geometry>
 <mesh filename="file://$(find gg_hex_description)/simple_hex/part_2.stl"/>
@@ -394,18 +394,18 @@
 </visual>
 <collision>
-<origin xyz="1.3877787807814456755e-17 0 0.14999999999999999445" rpy="3.141592653589793116 -4.3645711874439094161e-32 -2.7440535728855418873e-17" />
-<geometry>
-<mesh filename="file://$(find gg_hex_description)/simple_hex/part_2.stl"/>
-</geometry>
-</collision>
-<inertial>
-<origin xyz="0.034589021054141862177 -0.0010936380280668997911 -0.012500000000000011102" rpy="0 0 0"/>
+<origin xyz="1.3877787807814456755e-17 -1.3877787807814456755e-17 0.14999999999999999445" rpy="-3.141592653589793116 1.7984046345965779156e-32 3.88627629426162707e-17" />
+<geometry>
+<mesh filename="file://$(find gg_hex_description)/simple_hex/part_2.stl"/>
+</geometry>
+</collision>
+<inertial>
+<origin xyz="0.034589021054141862177 -0.0010936380280669110669 -0.012500000000000011102" rpy="0 0 0"/>
 <mass value="0.071677002780848500518" />
-<inertia ixx="8.7482057934132196188e-06" ixy="3.4865457641769578704e-06"  ixz="-1.9662530732822710513e-36" iyy="5.9817560075328712107e-05" iyz="-2.8818418605395030131e-36" izz="6.1300877458863529458e-05" />
+<inertia ixx="8.7482057934132196188e-06" ixy="3.4865457641769654937e-06"  ixz="-6.1910131917809796897e-36" iyy="5.9817560075328671449e-05" iyz="2.2131024314071804434e-35" izz="6.1300877458863529458e-05" />
 </inertial>
 </link>
 <link name="part_3_4">
 <visual>
-<origin xyz="-0.094999999999999987232 0.16249999999999995004 -0.02999999999999999889" rpy="1.570796326794896558 -8.0332321119309803377e-18 -4.1927494471144480461e-18" />
+<origin xyz="-0.095000000000000014988 0.1624999999999999778 -0.02999999999999999889" rpy="1.570796326794896558 5.3235004828166924622e-17 -1.6538240715905895521e-18" />
 <geometry>
 <mesh filename="file://$(find gg_hex_description)/simple_hex/part_3.stl"/>
@@ -416,18 +416,18 @@
 </visual>
 <collision>
-<origin xyz="-0.094999999999999987232 0.16249999999999995004 -0.02999999999999999889" rpy="1.570796326794896558 -8.0332321119309803377e-18 -4.1927494471144480461e-18" />
-<geometry>
-<mesh filename="file://$(find gg_hex_description)/simple_hex/part_3.stl"/>
-</geometry>
-</collision>
-<inertial>
-<origin xyz="0.037501640681764994434 2.7755575615628913511e-17 -0.0029167993347438475257" rpy="0 0 0"/>
-<mass value="0.053756066729807983062" />
-<inertia ixx="6.1725657961057495281e-06" ixy="-1.1803748872230270229e-22"  ixz="4.04222708638514997e-10" iyy="3.4211476506187103079e-05" iyz="3.5425208560944027467e-23" izz="3.3235315244488719284e-05" />
+<origin xyz="-0.095000000000000014988 0.1624999999999999778 -0.02999999999999999889" rpy="1.570796326794896558 5.3235004828166924622e-17 -1.6538240715905895521e-18" />
+<geometry>
+<mesh filename="file://$(find gg_hex_description)/simple_hex/part_3.stl"/>
+</geometry>
+</collision>
+<inertial>
+<origin xyz="0.037501640681764966678 0 -0.0029167993347438518625" rpy="0 0 0"/>
+<mass value="0.053756066729807990001" />
+<inertia ixx="6.1725657961057495281e-06" ixy="-2.1683971723577301091e-22"  ixz="4.0422270864038747541e-10" iyy="3.4211476506187116632e-05" iyz="-1.4047305842135536174e-23" izz="3.3235315244488732836e-05" />
 </inertial>
 </link>
 <link name="part_4_4">
 <visual>
-<origin xyz="-0.18249999999999994005 -0.1624999999999999778 0" rpy="-1.570796326794896558 2.8566655802302188636e-17 8.7504359132012681067e-19" />
+<origin xyz="-0.1824999999999999678 -0.1624999999999999778 -1.3877787807814456755e-17" rpy="-1.570796326794896558 -3.3524980809654333908e-18 8.7412952972356542727e-19" />
 <geometry>
 <mesh filename="file://$(find gg_hex_description)/simple_hex/part_4.stl"/>
@@ -438,18 +438,18 @@
 </visual>
 <collision>
-<origin xyz="-0.18249999999999994005 -0.1624999999999999778 0" rpy="-1.570796326794896558 2.8566655802302188636e-17 8.7504359132012681067e-19" />
-<geometry>
-<mesh filename="file://$(find gg_hex_description)/simple_hex/part_4.stl"/>
-</geometry>
-</collision>
-<inertial>
-<origin xyz="0.037500919815065564267 0 1.8396301308768877993e-07" rpy="0 0 0"/>
-<mass value="0.053754736812063892704" />
-<inertia ixx="6.6298075152166937701e-06" ixy="2.6044003590142730321e-22"  ixz="-5.3411963924549763738e-06" iyy="3.4666848127693282542e-05" iyz="-4.4995162169914313127e-23" izz="3.3233445124738749895e-05" />
+<origin xyz="-0.1824999999999999678 -0.1624999999999999778 -1.3877787807814456755e-17" rpy="-1.570796326794896558 -3.3524980809654333908e-18 8.7412952972356542727e-19" />
+<geometry>
+<mesh filename="file://$(find gg_hex_description)/simple_hex/part_4.stl"/>
+</geometry>
+</collision>
+<inertial>
+<origin xyz="0.037500919815065508756 0 1.839630130807241574e-07" rpy="0 0 0"/>
+<mass value="0.053754736812063899642" />
+<inertia ixx="6.629807515216692076e-06" ixy="1.3418374311804968992e-22"  ixz="-5.3411963924549789149e-06" iyy="3.4666848127693275766e-05" iyz="-3.4765513030092073148e-23" izz="3.3233445124738763448e-05" />
 </inertial>
 </link>
 <link name="part_5_4">
 <visual>
-<origin xyz="-0.27000000000000007327 -0.16249999999999995004 -0.029999999999999985012" rpy="-1.570796326794896558 -1.9707028344597000075e-17 1.0926112924473921313e-17" />
+<origin xyz="-0.27000000000000012879 -0.1624999999999999778 -0.030000000000000026645" rpy="-1.570796326794896558 1.0328680665792166888e-17 -2.1377999918909134721e-18" />
 <geometry>
 <mesh filename="file://$(find gg_hex_description)/simple_hex/part_5.stl"/>
@@ -460,17 +460,17 @@
 </visual>
 <collision>
-<origin xyz="-0.27000000000000007327 -0.16249999999999995004 -0.029999999999999985012" rpy="-1.570796326794896558 -1.9707028344597000075e-17 1.0926112924473921313e-17" />
-<geometry>
-<mesh filename="file://$(find gg_hex_description)/simple_hex/part_5.stl"/>
-</geometry>
-</collision>
-<inertial>
-<origin xyz="0.038984534277943516667 2.7755575615628913511e-17 -0.0013659706120265082373" rpy="0 0 0"/>
+<origin xyz="-0.27000000000000012879 -0.1624999999999999778 -0.030000000000000026645" rpy="-1.570796326794896558 1.0328680665792166888e-17 -2.1377999918909134721e-18" />
+<geometry>
+<mesh filename="file://$(find gg_hex_description)/simple_hex/part_5.stl"/>
+</geometry>
+</collision>
+<inertial>
+<origin xyz="0.038984534277943461156 0 -0.0013659706120265550748" rpy="0 0 0"/>
 <mass value="0.057365949134959140499" />
-<inertia ixx="6.7866051749620285596e-06" ixy="9.6615030819636046522e-22"  ixz="-2.7857025297757687092e-06" iyy="3.6471388191653054305e-05" iyz="-1.7067401810588130451e-21" izz="3.4867176458850274992e-05" />
+<inertia ixx="6.7866051749620285596e-06" ixy="1.9439685741526689876e-22"  ixz="-2.7857025297757716738e-06" iyy="3.6471388191653054305e-05" iyz="2.9170416666277988371e-24" izz="3.4867176458850274992e-05" />
 </inertial>
 </link>
 <joint name="joint1r2" type="revolute">
-<origin xyz="0.075000000000000122125 6.9388939039072283776e-18 -1.3877787807814456755e-17" rpy="-2.0733237872270123589e-15 1.0980092865848006522e-15 -1.3140831922292772749" />
+<origin xyz="0.075000000000000177636 -1.3877787807814456755e-17 -4.1633363423443370266e-17" rpy="-5.0325744217438855405e-15 1.0692776029102249568e-15 -3.2850944049226743711e-16" />
 <parent link="part_4_4" />
 <child link="part_5_4" />
@@ -480,5 +480,5 @@
 </joint>
 <joint name="joint2r2" type="revolute">
-<origin xyz="0.074999999999999816813 -2.3592239273284576484e-16 1.6653345369377348106e-16" rpy="3.1415926535897904515 1.8393475156992125372e-16 1.2898524636894628095e-15" />
+<origin xyz="0.075000000000000011102 2.0816681711721685133e-17 -2.7755575615628913511e-17" rpy="-3.141592653589793116 -6.5800803597219166288e-16 -2.9325568039305312645e-15" />
 <parent link="part_3_4" />
 <child link="part_4_4" />
@@ -488,5 +488,5 @@
 </joint>
 <joint name="joint3r2" type="revolute">
-<origin xyz="0.08249999999999997613 0 -0.012500000000000101308" rpy="1.5707963267948956698 -0.022955255919808830595 -1.1707595574204076793e-15" />
+<origin xyz="0.082500000000000073275 -2.7755575615628913511e-17 -0.012500000000000011102" rpy="1.5707963267948974462 -0.022955255919813049442 4.8869636822199225657e-17" />
 <parent link="part_2_4" />
 <child link="part_3_4" />
@@ -496,5 +496,5 @@
 </joint>
 <joint name="joint4r2" type="revolute">
-<origin xyz="-0.075000000000000011102 -0.12500000000000005551 0.035699999999999981748" rpy="-3.1415926535897917837 8.5540509271527851515e-17 -2.7052603405912107881" />
+<origin xyz="-0.074999999999995251021 -0.12499999999999757139 0.035699999999999107447" rpy="-3.1415926535897917837 8.5540509271467848783e-17 -2.7052603405911836987" />
 <parent link="part_6" />
 <child link="part_2_4" />
@@ -542,7 +542,7 @@
 </collision>
 <inertial>
-<origin xyz="0.037501640681765022189 5.5511151231257827021e-17 -0.0029167993347438405868" rpy="0 0 0"/>
-<mass value="0.053756066729807983062" />
-<inertia ixx="6.1725657961057529163e-06" ixy="3.8882305442281982282e-23"  ixz="4.0422270864018910716e-10" iyy="3.4211476506187116632e-05" iyz="1.8324368501750596821e-23" izz="3.3235315244488719284e-05" />
+<origin xyz="0.037501640681765022189 2.7755575615628913511e-17 -0.0029167993347438405868" rpy="0 0 0"/>
+<mass value="0.053756066729807990001" />
+<inertia ixx="6.1725657961057529163e-06" ixy="3.8882305442281982282e-23"  ixz="4.0422270864018915886e-10" iyy="3.4211476506187116632e-05" iyz="1.8324368501750596821e-23" izz="3.3235315244488719284e-05" />
 </inertial>
 </link>
@@ -564,12 +564,12 @@
 </collision>
 <inertial>
-<origin xyz="0.037500919815065508756 -2.7755575615628913511e-17 1.8396301309691188346e-07" rpy="0 0 0"/>
-<mass value="0.053754736812063892704" />
-<inertia ixx="6.6298075152166937701e-06" ixy="-4.6056281295966211398e-22"  ixz="-5.3411963924549780679e-06" iyy="3.4666848127693268989e-05" iyz="-6.394915084081913103e-23" izz="3.3233445124738763448e-05" />
+<origin xyz="0.037500919815065508756 -2.7755575615628913511e-17 1.8396301309692821531e-07" rpy="0 0 0"/>
+<mass value="0.053754736812063899642" />
+<inertia ixx="6.6298075152166937701e-06" ixy="-4.6056281295966201994e-22"  ixz="-5.3411963924549780679e-06" iyy="3.4666848127693262213e-05" iyz="-6.394915084081913103e-23" izz="3.3233445124738763448e-05" />
 </inertial>
 </link>
 <link name="part_5_5">
 <visual>
-<origin xyz="-0.27000000000000007327 -0.16249999999999992228 -0.029999999999999988481" rpy="-1.570796326794896558 2.8624636829500254542e-18 1.8983277563026202975e-17" />
+<origin xyz="-0.27000000000000007327 -0.1624999999999999778 -0.030000000000000002359" rpy="-1.570796326794896558 9.8708462230034056968e-18 -1.0354669235972614879e-17" />
 <geometry>
 <mesh filename="file://$(find gg_hex_description)/simple_hex/part_5.stl"/>
@@ -580,17 +580,17 @@
 </visual>
 <collision>
-<origin xyz="-0.27000000000000007327 -0.16249999999999992228 -0.029999999999999988481" rpy="-1.570796326794896558 2.8624636829500254542e-18 1.8983277563026202975e-17" />
-<geometry>
-<mesh filename="file://$(find gg_hex_description)/simple_hex/part_5.stl"/>
-</geometry>
-</collision>
-<inertial>
-<origin xyz="0.038984534277943565239 2.7755575615628913511e-17 -0.0013659706120265143088" rpy="0 0 0"/>
+<origin xyz="-0.27000000000000007327 -0.1624999999999999778 -0.030000000000000002359" rpy="-1.570796326794896558 9.8708462230034056968e-18 -1.0354669235972614879e-17" />
+<geometry>
+<mesh filename="file://$(find gg_hex_description)/simple_hex/part_5.stl"/>
+</geometry>
+</collision>
+<inertial>
+<origin xyz="0.038984534277943565239 -2.7755575615628913511e-17 -0.0013659706120265342581" rpy="0 0 0"/>
 <mass value="0.057365949134959140499" />
-<inertia ixx="6.7866051749620319477e-06" ixy="-2.5955244803830137033e-21"  ixz="-2.7857025297757691327e-06" iyy="3.6471388191653040752e-05" iyz="-4.4799247184293611423e-23" izz="3.4867176458850261439e-05" />
+<inertia ixx="6.7866051749620319477e-06" ixy="-1.6353903606745196843e-22"  ixz="-2.7857025297757682857e-06" iyy="3.6471388191653040752e-05" iyz="4.2286751152048867467e-23" izz="3.4867176458850261439e-05" />
 </inertial>
 </link>
 <joint name="joint1r1" type="revolute">
-<origin xyz="0.075000000000000066613 0 5.2041704279304212832e-18" rpy="-2.299179047061970185e-15 1.5362019183893119331e-15 -0.84638527925003248509" />
+<origin xyz="0.075000000000000122125 -1.3877787807814456755e-17 -1.7347234759768070944e-18" rpy="-8.8004447424903784714e-15 3.4050601472399260968e-15 1.0831047477735382302e-15" />
 <parent link="part_4_5" />
 <child link="part_5_5" />
@@ -662,7 +662,7 @@
 </collision>
 <inertial>
-<origin xyz="0.037501640681765036067 2.7755575615628913511e-17 -0.0029167993347438431889" rpy="0 0 0"/>
-<mass value="0.053756066729807983062" />
-<inertia ixx="6.1725657961057529163e-06" ixy="-2.1455208118593170949e-22"  ixz="4.0422270864188425873e-10" iyy="3.4211476506187116632e-05" iyz="-3.7935518535677754894e-23" izz="3.3235315244488732836e-05" />
+<origin xyz="0.037501640681765036067 0 -0.0029167993347438436226" rpy="0 0 0"/>
+<mass value="0.053756066729807990001" />
+<inertia ixx="6.1725657961057529163e-06" ixy="-2.1455208118593170949e-22"  ixz="4.0422270864188431043e-10" iyy="3.4211476506187116632e-05" iyz="-3.7935518535677754894e-23" izz="3.3235315244488732836e-05" />
 </inertial>
 </link>
@@ -684,12 +684,12 @@
 </collision>
 <inertial>
-<origin xyz="0.037500919815065481 0 1.8396301310265947846e-07" rpy="0 0 0"/>
-<mass value="0.053754736812063892704" />
-<inertia ixx="6.6298075152166903819e-06" ixy="-7.5178032060141378788e-23"  ixz="-5.3411963924549729857e-06" iyy="3.4666848127693282542e-05" iyz="7.0308005378485341663e-23" izz="3.3233445124738763448e-05" />
+<origin xyz="0.037500919815065487939 0 1.8396301310267578385e-07" rpy="0 0 0"/>
+<mass value="0.053754736812063899642" />
+<inertia ixx="6.6298075152166903819e-06" ixy="-7.5178032060141367033e-23"  ixz="-5.3411963924549729857e-06" iyy="3.4666848127693275766e-05" iyz="7.0308005378485341663e-23" izz="3.3233445124738763448e-05" />
 </inertial>
 </link>
 <link name="part_5_6">
 <visual>
-<origin xyz="-0.27000000000000012879 -0.16250000000000000555 -0.030000000000000012768" rpy="-1.570796326794896558 1.4856807686997467659e-18 2.6563038756197870876e-18" />
+<origin xyz="-0.27000000000000007327 -0.1624999999999999778 -0.030000000000000026645" rpy="-1.570796326794896558 -5.3587668691016062517e-17 -2.129463941218227213e-18" />
 <geometry>
 <mesh filename="file://$(find gg_hex_description)/simple_hex/part_5.stl"/>
@@ -700,17 +700,17 @@
 </visual>
 <collision>
-<origin xyz="-0.27000000000000012879 -0.16250000000000000555 -0.030000000000000012768" rpy="-1.570796326794896558 1.4856807686997467659e-18 2.6563038756197870876e-18" />
-<geometry>
-<mesh filename="file://$(find gg_hex_description)/simple_hex/part_5.stl"/>
-</geometry>
-</collision>
-<inertial>
-<origin xyz="0.038984534277943516667 -2.7755575615628913511e-17 -0.0013659706120265396791" rpy="0 0 0"/>
+<origin xyz="-0.27000000000000007327 -0.1624999999999999778 -0.030000000000000026645" rpy="-1.570796326794896558 -5.3587668691016062517e-17 -2.129463941218227213e-18" />
+<geometry>
+<mesh filename="file://$(find gg_hex_description)/simple_hex/part_5.stl"/>
+</geometry>
+</collision>
+<inertial>
+<origin xyz="0.038984534277943461156 -2.7755575615628913511e-17 -0.0013659706120265355592" rpy="0 0 0"/>
 <mass value="0.057365949134959140499" />
-<inertia ixx="6.7866051749620319477e-06" ixy="1.332064536689751159e-23"  ixz="-2.7857025297757687092e-06" iyy="3.6471388191653054305e-05" iyz="-1.5080345018492446682e-21" izz="3.4867176458850274992e-05" />
+<inertia ixx="6.7866051749620268655e-06" ixy="6.9281392874588607097e-23"  ixz="-2.7857025297757653211e-06" iyy="3.6471388191653040752e-05" iyz="1.8171849861395137679e-23" izz="3.4867176458850274992e-05" />
 </inertial>
 </link>
 <joint name="joint1r" type="revolute">
-<origin xyz="0.075000000000000011102 -6.9388939039072283776e-18 9.7144514654701197287e-17" rpy="-2.856431244057671654e-15 1.8673695075199355997e-15 -1.6742979852404027419" />
+<origin xyz="0.075000000000000011102 4.8572257327350598644e-17 2.7755575615628913511e-17" rpy="-7.7548675240533371154e-15 3.1532980223334467555e-15 1.3270558726469407914e-15" />
 <parent link="part_4_6" />
 <child link="part_5_6" />
