Commit message: spider_free_from_origin

File: install/gg_hex_description/share/gg_hex_description/simple_hex/robot.urdf.xacro (robot description, xacro)
@@ -1,4 +1,5 @@
 <?xml version="1.0"?>
 <robot name="gg_hex"  xmlns:xacro= "http://www.ros.org/wiki/xacro">
+<pose>0 0 0 0 0 0</pose>
 <link name="part_6">
 <visual>
@@ -743,10 +744,10 @@
 <joint_properties friction="0.0"/>
 </joint>
-<link name="world"/>
+<!-- <link name="world"/>
 <joint name="joint0" type="fixed">
 <origin xyz="0.0 0.0 0.25" rpy="0.0 0.0 0.0" />
   <parent link="world"/>
   <child link="part_6"/>
-  <pose>0 0 0 0 0 0</pose> <!-- Set the z-axis to 0.5 meters -->
-</joint>
+  <pose>0 0 0 0 0 0</pose>
+</joint> -->
 </robot>

Commit message: controller_dn

File: install/gg_hex_description/share/gg_hex_description/simple_hex/robot.urdf.xacro (robot description, xacro)
@@ -744,5 +744,5 @@
 <joint_properties friction="0.0"/>
 </joint>
-<!-- <link name="world"/>
+<link name="world"/>
 <joint name="joint0" type="fixed">
 <origin xyz="0.0 0.0 0.25" rpy="0.0 0.0 0.0" />
@@ -750,4 +750,4 @@
   <child link="part_6"/>
   <pose>0 0 0 0 0 0</pose>
-</joint> -->
+</joint>
 </robot>

File: src/gg_hex_description/simple_hex/robot_aditya.urdf.xacro (robot description, xacro)
@@ -1,5 +1,5 @@
 <?xml version="1.0"?>
 <robot name="gg_hex"  xmlns:xacro= "http://www.ros.org/wiki/xacro">
-<pose>0 0 0 0 0 0</pose>
+<!-- <pose>0 0 0 0 0 0</pose> -->
 <link name="part_6">
 <visual>
@@ -20,6 +20,6 @@
 <inertial>
 <origin xyz="0 -6.9388939039072283776e-18 0.023199999999999998401" rpy="0 0 0"/>
-<mass value="0.59529549486301092109" />
-<inertia ixx="0.0030748925185440614989" ixy="0"  ixz="0" iyy="0.0016906840458352414419" iyz="0" izz="0.0047035666169977386614" />
+<mass value="10.59529549486301092109" />
+<inertia ixx="10.0030748925185440614989" ixy="0"  ixz="0" iyy="10.0016906840458352414419" iyz="0" izz="10.0047035666169977386614" />
 </inertial>
 </link>
@@ -42,6 +42,6 @@
 <inertial>
 <origin xyz="0.034589021054141862177 -0.001093638028066900008 -0.012499999999999983347" rpy="0 0 0"/>
-<mass value="0.071677002780848500518" />
-<inertia ixx="8.7482057934132196188e-06" ixy="3.4865457641769595645e-06"  ixz="-1.4923544699764620014e-35" iyy="5.9817560075328685002e-05" iyz="4.7600900158112267165e-35" izz="6.1300877458863502352e-05" />
+<mass value="10.071677002780848500518" />
+<inertia ixx="18.7482057934132196188e-06" ixy="13.4865457641769595645e-06"  ixz="-11.4923544699764620014e-35" iyy="15.9817560075328685002e-05" iyz="4.7600900158112267165e-35" izz="6.1300877458863502352e-05" />
 </inertial>
 </link>
@@ -64,6 +64,6 @@
 <inertial>
 <origin xyz="0.0375016406817649528 0 -0.0029167993347438657403" rpy="0 0 0"/>
-<mass value="0.053756066729807990001" />
-<inertia ixx="6.1725657961057495281e-06" ixy="-3.9013430001076611365e-36"  ixz="4.0422270863664960132e-10" iyy="3.4211476506187116632e-05" iyz="4.0371463405644450255e-36" izz="3.3235315244488732836e-05" />
+<mass value="10.053756066729807990001" />
+<inertia ixx="16.1725657961057495281e-06" ixy="-13.9013430001076611365e-36"  ixz="14.0422270863664960132e-10" iyy="13.4211476506187116632e-05" iyz="4.0371463405644450255e-36" izz="3.3235315244488732836e-05" />
 </inertial>
 </link>
@@ -86,6 +86,6 @@
 <inertial>
 <origin xyz="0.037500919815065453244 0 1.8396301309196947268e-07" rpy="0 0 0"/>
-<mass value="0.053754736812063899642" />
-<inertia ixx="6.629807515216692076e-06" ixy="1.6458832113731393079e-38"  ixz="-5.3411963924549780679e-06" iyy="3.4666848127693275766e-05" iyz="-1.0240845939341500988e-37" izz="3.3233445124738763448e-05" />
+<mass value="10.053754736812063899642" />
+<inertia ixx="16.629807515216692076e-06" ixy="11.6458832113731393079e-38"  ixz="-15.3411963924549780679e-06" iyy="13.4666848127693275766e-05" iyz="-1.0240845939341500988e-37" izz="3.3233445124738763448e-05" />
 </inertial>
 </link>
@@ -108,6 +108,6 @@
 <inertial>
 <origin xyz="0.038984534277943398706 0 -0.0013659706120265383781" rpy="0 0 0"/>
-<mass value="0.057365949134959140499" />
-<inertia ixx="6.7866051749620268655e-06" ixy="-2.3680935053173413778e-36"  ixz="-2.7857025297757678622e-06" iyy="3.6471388191653054305e-05" iyz="1.9541077328988703576e-35" izz="3.4867176458850274992e-05" />
+<mass value="10.057365949134959140499" />
+<inertia ixx="16.7866051749620268655e-06" ixy="-12.3680935053173413778e-36"  ixz="-12.7857025297757678622e-06" iyy="13.6471388191653054305e-05" iyz="1.9541077328988703576e-35" izz="3.4867176458850274992e-05" />
 </inertial>
 </link>
@@ -162,6 +162,6 @@
 <inertial>
 <origin xyz="0.034589021054141848299 -0.0010936380280668978396 -0.012499999999999983347" rpy="0 0 0"/>
-<mass value="0.071677002780848500518" />
-<inertia ixx="8.7482057934132196188e-06" ixy="3.4865457641769612585e-06"  ixz="0" iyy="5.9817560075328685002e-05" iyz="0" izz="6.1300877458863502352e-05" />
+<mass value="10.071677002780848500518" />
+<inertia ixx="18.7482057934132196188e-06" ixy="13.4865457641769612585e-06"  ixz="0" iyy="15.9817560075328685002e-05" iyz="0" izz="16.1300877458863502352e-05" />
 </inertial>
 </link>
@@ -184,6 +184,6 @@
 <inertial>
 <origin xyz="0.037501640681764966678 0 -0.0029167993347438449236" rpy="0 0 0"/>
-<mass value="0.053756066729807990001" />
-<inertia ixx="6.1725657961057495281e-06" ixy="0"  ixz="4.0422270863981542832e-10" iyy="3.4211476506187116632e-05" iyz="0" izz="3.3235315244488732836e-05" />
+<mass value="10.053756066729807990001" />
+<inertia ixx="16.1725657961057495281e-06" ixy="0"  ixz="14.0422270863981542832e-10" iyy="13.4211476506187116632e-05" iyz="0" izz="13.3235315244488732836e-05" />
 </inertial>
 </link>
@@ -206,6 +206,6 @@
 <inertial>
 <origin xyz="0.037500919815065487939 0 1.8396301309581211706e-07" rpy="0 0 0"/>
-<mass value="0.053754736812063899642" />
-<inertia ixx="6.6298075152166937701e-06" ixy="0"  ixz="-5.3411963924549780679e-06" iyy="3.4666848127693275766e-05" iyz="0" izz="3.3233445124738763448e-05" />
+<mass value="10.053754736812063899642" />
+<inertia ixx="16.6298075152166937701e-06" ixy="0"  ixz="-15.3411963924549780679e-06" iyy="13.4666848127693275766e-05" iyz="0" izz="13.3233445124738763448e-05" />
 </inertial>
 </link>
@@ -228,6 +228,6 @@
 <inertial>
 <origin xyz="0.038984534277943565239 0 -0.001365970612026520814" rpy="0 0 0"/>
-<mass value="0.057365949134959140499" />
-<inertia ixx="6.7866051749620285596e-06" ixy="-1.0663918689120664312e-36"  ixz="-2.7857025297757682857e-06" iyy="3.6471388191653054305e-05" iyz="1.3555009886619676805e-35" izz="3.4867176458850274992e-05" />
+<mass value="10.057365949134959140499" />
+<inertia ixx="16.7866051749620285596e-06" ixy="-11.0663918689120664312e-36"  ixz="-12.7857025297757682857e-06" iyy="13.6471388191653054305e-05" iyz="1.3555009886619676805e-35" izz="3.4867176458850274992e-05" />
 </inertial>
 </link>
@@ -282,6 +282,6 @@
 <inertial>
 <origin xyz="0.034589021054141820544 -0.0010936380280669156205 -0.012499999999999983347" rpy="0 0 0"/>
-<mass value="0.071677002780848500518" />
-<inertia ixx="8.7482057934132196188e-06" ixy="3.4865457641769578704e-06"  ixz="0" iyy="5.9817560075328685002e-05" iyz="0" izz="6.1300877458863502352e-05" />
+<mass value="10.071677002780848500518" />
+<inertia ixx="18.7482057934132196188e-06" ixy="13.4865457641769578704e-06"  ixz="0" iyy="15.9817560075328685002e-05" iyz="0" izz="16.1300877458863502352e-05" />
 </inertial>
 </link>
@@ -304,6 +304,6 @@
 <inertial>
 <origin xyz="0.037501640681764980556 0 -0.0029167993347438440563" rpy="0 0 0"/>
-<mass value="0.053756066729807990001" />
-<inertia ixx="6.1725657961057495281e-06" ixy="3.3866754089596615417e-36"  ixz="4.042227086378963176e-10" iyy="3.4211476506187116632e-05" iyz="-4.9525034835553173072e-36" izz="3.3235315244488732836e-05" />
+<mass value="10.053756066729807990001" />
+<inertia ixx="16.1725657961057495281e-06" ixy="13.3866754089596615417e-36"  ixz="14.042227086378963176e-10" iyy="13.4211476506187116632e-05" iyz="-14.9525034835553173072e-36" izz="13.3235315244488732836e-05" />
 </inertial>
 </link>
@@ -326,6 +326,6 @@
 <inertial>
 <origin xyz="0.037500919815065487939 0 1.8396301310722493311e-07" rpy="0 0 0"/>
-<mass value="0.053754736812063899642" />
-<inertia ixx="6.629807515216692076e-06" ixy="8.4076706020862930361e-36"  ixz="-5.3411963924549780679e-06" iyy="3.4666848127693275766e-05" iyz="-5.2557119676207727929e-36" izz="3.3233445124738763448e-05" />
+<mass value="10.053754736812063899642" />
+<inertia ixx="16.629807515216692076e-06" ixy="18.4076706020862930361e-36"  ixz="-15.3411963924549780679e-06" iyy="13.4666848127693275766e-05" iyz="-15.2557119676207727929e-36" izz="13.3233445124738763448e-05" />
 </inertial>
 </link>
@@ -348,6 +348,6 @@
 <inertial>
 <origin xyz="0.038984534277943565239 0 -0.0013659706120265464012" rpy="0 0 0"/>
-<mass value="0.057365949134959140499" />
-<inertia ixx="6.7866051749620285596e-06" ixy="1.1415885784153511439e-35"  ixz="-2.7857025297757670152e-06" iyy="3.6471388191653054305e-05" iyz="9.8847353391390472314e-36" izz="3.4867176458850274992e-05" />
+<mass value="10.057365949134959140499" />
+<inertia ixx="16.7866051749620285596e-06" ixy="11.1415885784153511439e-35"  ixz="-12.7857025297757670152e-06" iyy="13.6471388191653054305e-05" iyz="19.8847353391390472314e-36" izz="13.4867176458850274992e-05" />
 </inertial>
 </link>
@@ -402,6 +402,6 @@
 <inertial>
 <origin xyz="0.034589021054141862177 -0.0010936380280669110669 -0.012500000000000011102" rpy="0 0 0"/>
-<mass value="0.071677002780848500518" />
-<inertia ixx="8.7482057934132196188e-06" ixy="3.4865457641769654937e-06"  ixz="-6.1910131917809796897e-36" iyy="5.9817560075328671449e-05" iyz="2.2131024314071804434e-35" izz="6.1300877458863529458e-05" />
+<mass value="10.071677002780848500518" />
+<inertia ixx="18.7482057934132196188e-06" ixy="13.4865457641769654937e-06"  ixz="-16.1910131917809796897e-36" iyy="15.9817560075328671449e-05" iyz="12.2131024314071804434e-35" izz="16.1300877458863529458e-05" />
 </inertial>
 </link>
@@ -424,6 +424,6 @@
 <inertial>
 <origin xyz="0.037501640681764966678 0 -0.0029167993347438518625" rpy="0 0 0"/>
-<mass value="0.053756066729807990001" />
-<inertia ixx="6.1725657961057495281e-06" ixy="-2.1683971723577301091e-22"  ixz="4.0422270864038747541e-10" iyy="3.4211476506187116632e-05" iyz="-1.4047305842135536174e-23" izz="3.3235315244488732836e-05" />
+<mass value="10.053756066729807990001" />
+<inertia ixx="16.1725657961057495281e-06" ixy="-12.1683971723577301091e-22"  ixz="14.0422270864038747541e-10" iyy="13.4211476506187116632e-05" iyz="-11.4047305842135536174e-23" izz="13.3235315244488732836e-05" />
 </inertial>
 </link>
@@ -446,6 +446,6 @@
 <inertial>
 <origin xyz="0.037500919815065508756 0 1.839630130807241574e-07" rpy="0 0 0"/>
-<mass value="0.053754736812063899642" />
-<inertia ixx="6.629807515216692076e-06" ixy="1.3418374311804968992e-22"  ixz="-5.3411963924549789149e-06" iyy="3.4666848127693275766e-05" iyz="-3.4765513030092073148e-23" izz="3.3233445124738763448e-05" />
+<mass value="10.053754736812063899642" />
+<inertia ixx="16.629807515216692076e-06" ixy="11.3418374311804968992e-22"  ixz="-15.3411963924549789149e-06" iyy="13.4666848127693275766e-05" iyz="-13.4765513030092073148e-23" izz="13.3233445124738763448e-05" />
 </inertial>
 </link>
@@ -468,6 +468,6 @@
 <inertial>
 <origin xyz="0.038984534277943461156 0 -0.0013659706120265550748" rpy="0 0 0"/>
-<mass value="0.057365949134959140499" />
-<inertia ixx="6.7866051749620285596e-06" ixy="1.9439685741526689876e-22"  ixz="-2.7857025297757716738e-06" iyy="3.6471388191653054305e-05" iyz="2.9170416666277988371e-24" izz="3.4867176458850274992e-05" />
+<mass value="10.057365949134959140499" />
+<inertia ixx="16.7866051749620285596e-06" ixy="11.9439685741526689876e-22"  ixz="-12.7857025297757716738e-06" iyy="13.6471388191653054305e-05" iyz="12.9170416666277988371e-24" izz="13.4867176458850274992e-05" />
 </inertial>
 </link>
@@ -522,6 +522,6 @@
 <inertial>
 <origin xyz="0.034589021054141848299 -0.0010936380280668976227 -0.012499999999999983347" rpy="0 0 0"/>
-<mass value="0.071677002780848500518" />
-<inertia ixx="8.7482057934132196188e-06" ixy="3.486545764176960835e-06"  ixz="-2.0212652133460496805e-37" iyy="5.9817560075328671449e-05" iyz="-5.8984668236420045281e-36" izz="6.1300877458863502352e-05" />
+<mass value="10.071677002780848500518" />
+<inertia ixx="18.7482057934132196188e-06" ixy="13.486545764176960835e-06"  ixz="-12.0212652133460496805e-37" iyy="15.9817560075328671449e-05" iyz="-15.8984668236420045281e-36" izz="16.1300877458863502352e-05" />
 </inertial>
 </link>
@@ -544,6 +544,6 @@
 <inertial>
 <origin xyz="0.037501640681765022189 2.7755575615628913511e-17 -0.0029167993347438405868" rpy="0 0 0"/>
-<mass value="0.053756066729807990001" />
-<inertia ixx="6.1725657961057529163e-06" ixy="3.8882305442281982282e-23"  ixz="4.0422270864018915886e-10" iyy="3.4211476506187116632e-05" iyz="1.8324368501750596821e-23" izz="3.3235315244488719284e-05" />
+<mass value="10.053756066729807990001" />
+<inertia ixx="16.1725657961057529163e-06" ixy="13.8882305442281982282e-23"  ixz="14.0422270864018915886e-10" iyy="13.4211476506187116632e-05" iyz="11.8324368501750596821e-23" izz="13.3235315244488719284e-05" />
 </inertial>
 </link>
@@ -566,6 +566,6 @@
 <inertial>
 <origin xyz="0.037500919815065508756 -2.7755575615628913511e-17 1.8396301309692821531e-07" rpy="0 0 0"/>
-<mass value="0.053754736812063899642" />
-<inertia ixx="6.6298075152166937701e-06" ixy="-4.6056281295966201994e-22"  ixz="-5.3411963924549780679e-06" iyy="3.4666848127693262213e-05" iyz="-6.394915084081913103e-23" izz="3.3233445124738763448e-05" />
+<mass value="10.053754736812063899642" />
+<inertia ixx="16.6298075152166937701e-06" ixy="-14.6056281295966201994e-22"  ixz="-15.3411963924549780679e-06" iyy="13.4666848127693262213e-05" iyz="-16.394915084081913103e-23" izz="13.3233445124738763448e-05" />
 </inertial>
 </link>
@@ -588,6 +588,6 @@
 <inertial>
 <origin xyz="0.038984534277943565239 -2.7755575615628913511e-17 -0.0013659706120265342581" rpy="0 0 0"/>
-<mass value="0.057365949134959140499" />
-<inertia ixx="6.7866051749620319477e-06" ixy="-1.6353903606745196843e-22"  ixz="-2.7857025297757682857e-06" iyy="3.6471388191653040752e-05" iyz="4.2286751152048867467e-23" izz="3.4867176458850261439e-05" />
+<mass value="10.057365949134959140499" />
+<inertia ixx="16.7866051749620319477e-06" ixy="-11.6353903606745196843e-22"  ixz="-12.7857025297757682857e-06" iyy="13.6471388191653040752e-05" iyz="14.2286751152048867467e-23" izz="13.4867176458850261439e-05" />
 </inertial>
 </link>
@@ -642,6 +642,6 @@
 <inertial>
 <origin xyz="0.034589021054141862177 -0.0010936380280668865639 -0.012499999999999983347" rpy="0 0 0"/>
-<mass value="0.071677002780848500518" />
-<inertia ixx="8.7482057934132196188e-06" ixy="3.486545764176959988e-06"  ixz="-1.07829961582057066e-37" iyy="5.9817560075328685002e-05" iyz="-4.2974994494111276226e-38" izz="6.1300877458863502352e-05" />
+<mass value="10.071677002780848500518" />
+<inertia ixx="18.7482057934132196188e-06" ixy="13.486545764176959988e-06"  ixz="-11.07829961582057066e-37" iyy="15.9817560075328685002e-05" iyz="-14.2974994494111276226e-38" izz="16.1300877458863502352e-05" />
 </inertial>
 </link>
@@ -664,6 +664,6 @@
 <inertial>
 <origin xyz="0.037501640681765036067 0 -0.0029167993347438436226" rpy="0 0 0"/>
-<mass value="0.053756066729807990001" />
-<inertia ixx="6.1725657961057529163e-06" ixy="-2.1455208118593170949e-22"  ixz="4.0422270864188431043e-10" iyy="3.4211476506187116632e-05" iyz="-3.7935518535677754894e-23" izz="3.3235315244488732836e-05" />
+<mass value="10.053756066729807990001" />
+<inertia ixx="16.1725657961057529163e-06" ixy="-12.1455208118593170949e-22"  ixz="14.0422270864188431043e-10" iyy="13.4211476506187116632e-05" iyz="-13.7935518535677754894e-23" izz="13.3235315244488732836e-05" />
 </inertial>
 </link>
@@ -686,6 +686,6 @@
 <inertial>
 <origin xyz="0.037500919815065487939 0 1.8396301310267578385e-07" rpy="0 0 0"/>
-<mass value="0.053754736812063899642" />
-<inertia ixx="6.6298075152166903819e-06" ixy="-7.5178032060141367033e-23"  ixz="-5.3411963924549729857e-06" iyy="3.4666848127693275766e-05" iyz="7.0308005378485341663e-23" izz="3.3233445124738763448e-05" />
+<mass value="10.053754736812063899642" />
+<inertia ixx="16.6298075152166903819e-06" ixy="-17.5178032060141367033e-23"  ixz="-15.3411963924549729857e-06" iyy="13.4666848127693275766e-05" iyz="17.0308005378485341663e-23" izz="13.3233445124738763448e-05" />
 </inertial>
 </link>
@@ -708,6 +708,6 @@
 <inertial>
 <origin xyz="0.038984534277943461156 -2.7755575615628913511e-17 -0.0013659706120265355592" rpy="0 0 0"/>
-<mass value="0.057365949134959140499" />
-<inertia ixx="6.7866051749620268655e-06" ixy="6.9281392874588607097e-23"  ixz="-2.7857025297757653211e-06" iyy="3.6471388191653040752e-05" iyz="1.8171849861395137679e-23" izz="3.4867176458850274992e-05" />
+<mass value="10.057365949134959140499" />
+<inertia ixx="16.7866051749620268655e-06" ixy="16.9281392874588607097e-23"  ixz="-12.7857025297757653211e-06" iyy="13.6471388191653040752e-05" iyz="11.8171849861395137679e-23" izz="13.4867176458850274992e-05" />
 </inertial>
 </link>
@@ -744,5 +744,5 @@
 <joint_properties friction="0.0"/>
 </joint>
-<link name="world"/>
+<!-- <link name="world"/>
 <joint name="joint0" type="fixed">
 <origin xyz="0.0 0.0 0.25" rpy="0.0 0.0 0.0" />
@@ -751,3 +751,4 @@
   <pose>0 0 0 0 0 0</pose>
 </joint>
+ -->
 </robot>
